File: Board.brd (EAGLE design)
At the start: 160 x 100 mm, 12 parts, among them K1 S102S02, K2 S102S02, Q1 310mA/60V/1.6Ω, Q2 310mA/60V/1.6Ω

Commit message: Work
Parts:
- removed K1, K2: S102S02, relay:S202S02
- removed R3, R4: (no value), resistor:M1206
- removed X1: (no value), con-subd:F25VP
- added C1, C2, C6: 10uF, resistor:C1206
- added C3, C5: 0.01uF, resistor:C1206
- added C4: (no value), resistor:C1206
- added IC1: BUF634U, burr-brown:SO08
- added IC2: LM555D, linear:SO08
- added PPSOUT, RUB_TEST_FREQ: BU-SMA-V, con-coax:BU-SMA-V
- added Q3: 35A/25V/8.5mΩ, SparkFun-DiscreteSemi:DPAK
- added RUBIDIUM: (no value), con-subd:F25VP
- added S1: (no value), switch:M9040P
- added TP1: PTR1PAD1-13, testpad:P1-13
- added U$3, U$4, U$5: MIC5014, FRC696:SOIC8
- added X3: MSTBV4, con-phoenix-508:MSTBV4
- Q1, Q2: value 310mA/60V/1.6Ω -> 35A/25V/8.5mΩ; device SparkFun-DiscreteSemi:SOT323 -> SparkFun-DiscreteSemi:DPAK
- R1: device resistor:M1206 -> resistor:R1206
- R2: value (none) -> 1k; device resistor:M1206 -> resistor:R1206
- moved Q2 83.6 mm to (-38.1, -30.5), turned to 0 degrees
- moved U$2 73.7 mm to (-29.2, -25.4)
- moved R2 48.3 mm to (82.5, 59.7)
- moved R1 42.7 mm to (67.3, 56.5), turned to 90 degrees
- moved U$1 12.6 mm to (52.1, 16.5), turned to 270 degrees
- moved Q1 8.13 mm to (43.2, 24.1), turned to 0 degrees
- moved X2 6.84 mm to (83.8, 6.35)
Connections:
- new net +24V: C6.1, Q2.4, U$5.1, X3.4
- new net CRYSTAL_HEAT: U$2.3, U$2.4
- new net GPS_PPS: S1.1
- new net N$10: Q2.1, U$5.5
- new net N$5: Q1.1, U$3.5
- new net N$6: C4.1, IC2.6, IC2.7, R1.1
- new net N$7: C3.1, IC2.5
- new net N$8: IC1.1, R2.1
- new net N$9: Q2.3, U$2.1, U$2.2, U$5.3
- new net RAWPPS: S1.2
- new net RUB_LOCK: RUBIDIUM.22
- new net RUB_PPS: RUBIDIUM.20, S1.3, TP1.TP
- new net RUB_TEST_FREQ: RUBIDIUM.23, RUB_TEST_FREQ.1
- net +15V: now also C1.1, Q1.4, U$3.1, X3.3; no longer K1.1
- net +5V: now also C2.1, C5.1, IC1.7, IC2.4, IC2.8, Q3.4, R1.2, U$4.1, X3.2; no longer K2.1
- net GND: now also C1.2, C2.2, C3.2, C4.2, C5.2, C6.2, IC1.4, IC2.1, PPSOUT.2, PPSOUT.3, PPSOUT.4, PPSOUT.5, R2.2, RUBIDIUM.1, RUBIDIUM.10, RUBIDIUM.14, RUBIDIUM.15, RUBIDIUM.19, RUBIDIUM.2, RUBIDIUM.21, RUBIDIUM.6, RUBIDIUM.7, RUBIDIUM.9, RUB_TEST_FREQ.2, RUB_TEST_FREQ.3, RUB_TEST_FREQ.4, RUB_TEST_FREQ.5, U$3.4, U$4.4, U$5.4, X3.1; no longer K1.4, K2.4, Q1.2, Q2.2, X1.1, X1.10, X1.14, X1.15, X1.19, X1.2, X1.21, X1.6, X1.7, X1.9
- net N$1: now also Q1.3, U$3.3; no longer K1.2
- net N$2: now also Q3.1, U$4.5; no longer K1.3, Q1.3, R1.1, R2.2
- net N$3: now also IC1.6, PPSOUT.1; no longer K2.2, U$2.1, U$2.2
- net N$4: now also IC1.3, IC2.3; no longer K2.3, Q2.3, R3.1, R4.2
- net RUBIDIUM_15: now also RUBIDIUM.16, RUBIDIUM.17, RUBIDIUM.18, RUBIDIUM.3, RUBIDIUM.4, RUBIDIUM.5; no longer R1.2, X1.16, X1.17, X1.18, X1.3, X1.4, X1.5
- net RUBIDIUM_5V: now also Q3.3, RUBIDIUM.8, U$4.3; no longer R3.2, U$2.3, U$2.4, X1.8
Routing:
- net +5V: track 0.00 -> 171.0 mm, vias 0 -> 1
- net +15V: track 0.00 -> 65.9 mm
- net RUB_PPS: track 0.00 -> 43.5 mm
- net RUBIDIUM_15: track 0.00 -> 27.4 mm
- net RUB_TEST_FREQ: track 0.00 -> 22.0 mm
- net RUBIDIUM_5V: track 0.00 -> 19.3 mm
- net N$5: track 0.00 -> 17.3 mm
- net N$2: track 0.00 -> 17.3 mm
- net N$1: track 0.00 -> 10.2 mm
- net N$6: track 0.00 -> 7.77 mm
- net N$3: track 0.00 -> 6.91 mm
- net N$4: track 0.00 -> 4.31 mm
- net N$8: track 0.00 -> 2.77 mm
- net N$7: track 0.00 -> 2.57 mm
Other:
- board size 160 x 100 mm -> 110.5 x 61 mm

Commit message: Schematic work
Parts:
- added U$6: PIC18F25K42SOIC, FRC696:SO28W
Connections:
- new net RUB_15_I: U$1.7
- net +5V: now also U$6.20
- net GND: now also U$6.19, U$6.8
Changed lines of the file:
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@@
 </element>
 <element name="C6" library="resistor" package="C1206" value="10uF" x="-30.48" y="-44.45"/>
+<element name="U$6" library="FRC696" package="SO28W" value="PIC18F25K42SOIC" x="45.72" y="46.99"/>
 </elements>
 <signals>
@@
 <contactref element="U$5" pad="4"/>
 <contactref element="C6" pad="2"/>
+<contactref element="U$6" pad="8"/>
+<contactref element="U$6" pad="19"/>
 <wire x1="90.1601" y1="57.1599" x2="95.2599" y2="57.1599" width="0" layer="19" extent="1-1"/>
 <wire x1="95.2599" y1="52.0601" x2="95.2599" y2="57.1599" width="0" layer="19" extent="1-1"/>
@@
 <wire x1="-29.08" y1="-44.45" x2="-27.305" y2="-22.7838" width="0" layer="19" extent="1-1"/>
 <wire x1="-36.195" y1="-49.59" x2="-29.08" y2="-44.45" width="0" layer="19" extent="1-1"/>
+<wire x1="48.895" y1="51.59" x2="-36.195" y2="-49.59" width="0" layer="19" extent="1-1"/>
+<wire x1="46.355" y1="42.39" x2="48.895" y2="51.59" width="0" layer="19" extent="1-1"/>
 </signal>
 <signal name="RUBIDIUM_15">
@@
 <wire x1="76.26" y1="62.805" x2="76.2" y2="62.865" width="0.4064" layer="1"/>
 <contactref element="U$2" pad="8"/>
+<contactref element="U$6" pad="20"/>
 <wire x1="58.42" y1="38.1" x2="71.06" y2="52.07" width="0" layer="19" extent="1-16"/>
 <wire x1="-31.115" y1="-22.7838" x2="25.4" y2="25.718" width="0" layer="19" extent="1-1"/>
+<wire x1="47.625" y1="51.59" x2="-31.115" y2="-22.7838" width="0" layer="19" extent="1-1"/>
 </signal>
 <signal name="RUB_LOCK">
@@
 <wire x1="13.97" y1="48.26" x2="-38.1" y2="-28.892" width="0" layer="19" extent="1-1"/>
 </signal>
+<signal name="RUB_15_I">
+<contactref element="U$1" pad="7"/>
+</signal>
 </signals>

Commit message: PCB work
Parts:
- added CRYSTAL: (no value), con-subd:F25VP
- added J1: RASPBERRYPI-40-PIN-GPIO_PTH_NO_SHROUD, SparkFun-Connectors:2X20
- added Q4: 220mA/50V/3.5Ω, SparkFun-DiscreteSemi:SOT23-3
- added R3: 1k, resistor:R1206
- moved X2 43.1 mm to (115.6, 35.6), turned to 90 degrees
- moved U$6 38.6 mm to (52.1, 85.1)
- moved IC2 22.2 mm to (85.1, 34.9)
- moved C4 22.2 mm to (76.2, 37.5)
- moved PPSOUT 22.2 mm to (104.1, 35.6)
- moved R2 22.2 mm to (94.0, 40.6)
- moved C3 22.2 mm to (83.8, 39.4)
- moved C5 22.2 mm to (72.4, 40.6)
- moved IC1 22.2 mm to (94.6, 36.2)
- moved R1 22.2 mm to (78.7, 37.5)
- moved RUB_TEST_FREQ 8.98 mm to (5.08, 19.1)
- moved X3 8.89 mm to (5.08, 40.6)
- moved RUBIDIUM 1.27 mm to (33.0, 6.35)
- moved S1 1.27 mm to (63.5, 22.9)
- moved TP1 1.27 mm to (63.5, 12.7)
Connections:
- new net 3.3V: J1.1, J1.17
- new net 5V: J1.2, J1.4
- new net N$11: IC2.2, Q4.3, R3.2
- net +5V: now also R3.1
- net GND: now also J1.14, J1.20, J1.25, J1.30, J1.34, J1.39, J1.6, J1.9, Q4.2
- net RAWPPS: now also Q4.1
Routing:
- net +5V: track 171.0 -> 196.3 mm
- net RAWPPS: track 0.00 -> 18.7 mm
- net N$11: track 0.00 -> 17.1 mm
- net +15V: track 65.9 -> 74.8 mm
- net RUB_TEST_FREQ: track 22.0 -> 29.1 mm
- net RUBIDIUM_15: track 27.4 -> 28.4 mm
- net RUBIDIUM_5V: track 19.3 -> 18.8 mm
Other:
- board size 110.5 x 61 mm -> 127 x 63.5 mm

Commit message: Adding crystal
Parts:
- added C7: 10uF, resistor:C1206
- added PPSOUT1: BU-SMA-V, con-coax:BU-SMA-V
- added Q5: 35A/25V/8.5mΩ, SparkFun-DiscreteSemi:DPAK
- added U$8: MIC5014, FRC696:SOIC8
- moved U$5 140.1 mm to (82.5, 24.1)
- moved C6 139.0 mm to (88.9, 26.7)
- moved Q2 125.5 mm to (74.9, 24.1)
- moved U$2 120.5 mm to (83.8, 16.5), turned to 270 degrees
- moved X2 6.35 mm to (120.7, 39.4)
Connections:
- removed net 5V: J1.2, J1.4
- new net CRYSTAL_EFC: CRYSTAL.5
- new net CRYSTAL_HEAT_EN: U$5.2
- new net CRYSTAL_HEAT_IMON: U$2.7
- new net CRYSTAL_LOGIC: CRYSTAL.15, Q5.3, U$8.3
- new net CRYSTAL_LOGIC_EN: U$8.2
- new net CRYSTAL_OUT: CRYSTAL.1, PPSOUT1.1
- new net CRYSTAL_OVEN_MON: CRYSTAL.9
- new net N$14: Q5.1, U$8.5
- net +24V: now also C7.1, Q5.4, U$8.1
- net +5V: now also J1.2, J1.4
- net CRYSTAL_HEAT: now also CRYSTAL.10, CRYSTAL.11, CRYSTAL.22, CRYSTAL.23
- net GND: now also C7.2, CRYSTAL.12, CRYSTAL.13, CRYSTAL.14, CRYSTAL.16, CRYSTAL.17, CRYSTAL.2, CRYSTAL.24, CRYSTAL.25, CRYSTAL.3, CRYSTAL.4, PPSOUT1.2, PPSOUT1.3, PPSOUT1.4, PPSOUT1.5, U$8.4
Routing:
- net +24V: track 0.00 -> 26.5 mm
- net CRYSTAL_LOGIC: track 0.00 -> 22.7 mm
- net CRYSTAL_OUT: track 0.00 -> 18.7 mm
- net CRYSTAL_HEAT: track 0.00 -> 18.4 mm
- net N$10: track 0.00 -> 17.3 mm
- net N$9: track 0.00 -> 10.2 mm
- net N$14: track 0.00 -> 6.28 mm
