File: Board.sch (EAGLE design)
At the start: 12 parts, among them K1 S102S02, K2 S102S02, Q1 310mA/60V/1.6Ω, Q2 310mA/60V/1.6Ω

Commit message: Work
Parts:
- removed K1, K2: S102S02, relay:S102S02
- removed R3, R4: (no value), resistor:R-US_M1206
- added C1, C2, C6: 10uF, resistor:C-EUC1206
- added C3, C5: 0.01uF, resistor:C-EUC1206
- added C4: (no value), resistor:C-EUC1206
- added IC1: BUF634U, burr-brown:BUF634U
- added IC2: LM555D, linear:LM555D
- added PPSOUT, RUB_TEST_FREQ: BU-SMA-V, con-coax:BU-SMA-V
- added Q3: 35A/25V/8.5mΩ, SparkFun-DiscreteSemi:MOSFET-NCH-FDD8780
- added S1: (no value), switch:M9040P
- added TP1: PTR1PAD1-13, testpad:PTR1PAD1-13
- added U$3, U$4, U$5: MIC5014, FRC696:MIC5014
- added X3: MSTBV4, con-phoenix-508:MSTBV4
- Q1, Q2: value 310mA/60V/1.6Ω -> 35A/25V/8.5mΩ; device SparkFun-DiscreteSemi:MOSFET-NCH-2N7002PW -> SparkFun-DiscreteSemi:MOSFET-NCH-FDD8780
- R1: device resistor:R-US_M1206 -> resistor:R-US_R1206
- R2: value (none) -> 1k; device resistor:R-US_M1206 -> resistor:R-US_R1206
- renumbered X1 to RUBIDIUM
Connections:
- new net +24V: C6.1, Q2.D, U$5.V+, X3-4.1
- new net CRYSTAL_HEAT: U$2.IP-@3, U$2.IP-@4
- new net GPS_PPS: S1.O
- new net N$10: Q2.G, U$5.GATE
- new net N$5: Q1.G, U$3.GATE
- new net N$6: C4.1, IC2.DIS, IC2.THR, R1.1
- new net N$7: C3.1, IC2.CV
- new net N$8: IC1.BW, R2.1
- new net N$9: Q2.S, U$2.IP+@1, U$2.IP+@2, U$5.SOURCE
- new net RAWPPS: S1.P
- new net RUB_LOCK: RUBIDIUM.22
- new net RUB_PPS: RUBIDIUM.20, S1.S, TP1.TP
- new net RUB_TEST_FREQ: RUBIDIUM.23, RUB_TEST_FREQ.1
- net +15V: now also C1.1, Q1.D, U$3.V+, X3-3.1; no longer K1.DS1
- net +5V: now also C2.1, C5.1, IC1.V+, IC2.R, IC2.V+, Q3.D, R1.2, U$4.V+, X3-2.1; no longer K2.DS1
- net GND: now also C1.2, C2.2, C3.2, C4.2, C5.2, C6.2, IC1.V-, IC2.GND, PPSOUT.2, R2.2, RUB_TEST_FREQ.2, U$3.GND, U$4.GND, U$5.GND, X3-1.1; no longer K1.K, K2.K, Q1.S, Q2.S
- net N$1: now also Q1.S, U$3.SOURCE; no longer K1.DS2
- net N$2: now also Q3.G, U$4.GATE; no longer K1.A, Q1.D, R1.1, R2.2
- net N$3: now also IC1.OUT, PPSOUT.1; no longer K2.DS2, U$2.IP+@1, U$2.IP+@2
- net N$4: now also IC1.IN, IC2.Q; no longer K2.A, Q2.D, R3.1, R4.2
- net RUBIDIUM_15: no longer R1.2
- net RUBIDIUM_5V: now also Q3.S, U$4.SOURCE; no longer R3.2, U$2.IP-@3, U$2.IP-@4

Commit message: Schematic work
Parts:
- added U$6: PIC18F25K42SOIC, FRC696:PIC18F25K42SOIC
Connections:
- new net RUB_15_I: U$1.VOUT
- net +5V: now also U$6.VDD
- net GND: now also U$6.VSS@1, U$6.VSS@2
Changed lines of the file:
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@@
 <part name="SUPPLY27" library="supply2" deviceset="+24V" device=""/>
 <part name="SUPPLY41" library="supply2" deviceset="+24V" device=""/>
+<part name="U$6" library="FRC696" deviceset="PIC18F25K42" device="SOIC"/>
+<part name="SUPPLY42" library="supply2" deviceset="+5V" device=""/>
+<part name="SUPPLY43" library="supply2" deviceset="GND" device=""/>
 </parts>
 <sheets>
@@
 </segment>
 </net>
+<net name="RUB_15_I" class="0">
+<segment>
+<pinref part="U$1" gate="G$1" pin="VOUT"/>
+<wire x1="86.36" y1="91.44" x2="86.36" y2="86.36" width="0.1524" layer="91"/>
+<label x="86.36" y="86.36" size="1.778" layer="95" rot="R270"/>
+</segment>
+</net>
 </nets>
 </sheet>
@@
 </segment>
 </net>
+</nets>
+</sheet>
+<sheet>
+<description>Microcontroller</description>
+<plain>
+</plain>
+<instances>
+<instance part="U$6" gate="G$1" x="63.5" y="63.5"/>
+<instance part="SUPPLY42" gate="+5V" x="63.5" y="88.9"/>
+<instance part="SUPPLY43" gate="GND" x="63.5" y="25.4"/>
+</instances>
+<busses>
+</busses>
+<nets>
+<net name="+5V" class="0">
+<segment>
+<pinref part="U$6" gate="G$1" pin="VDD"/>
+<pinref part="SUPPLY42" gate="+5V" pin="+5V"/>
+</segment>
+</net>
+<net name="GND" class="0">
+<segment>
+<pinref part="U$6" gate="G$1" pin="VSS@1"/>
+<pinref part="SUPPLY43" gate="GND" pin="GND"/>
+<wire x1="60.96" y1="27.94" x2="63.5" y2="27.94" width="0.1524" layer="91"/>
+<pinref part="U$6" gate="G$1" pin="VSS@2"/>
+<wire x1="63.5" y1="27.94" x2="66.04" y2="27.94" width="0.1524" layer="91"/>
+<junction x="63.5" y="27.94"/>
+</segment>
+</net>

Commit message: PCB work
Parts:
- added CRYSTAL: (no value), con-subd:F25VP
- added J1: RASPBERRYPI-40-PIN-GPIO_PTH_NO_SHROUD, SparkFun-Connectors:RASPBERRYPI-40-PIN-GPIO_PTH_NO_SHROUD
- added Q4: 220mA/50V/3.5Ω, SparkFun-DiscreteSemi:MOSFET-NCH-BSS138
- added R3: 1k, resistor:R-US_R1206
Connections:
- new net N$11: IC2.TR, Q4.D, R3.2
- net +5V: now also R3.1
- net GND: now also Q4.S
- net RAWPPS: now also Q4.G
Changed lines of the file:
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@@
 <part name="SUPPLY42" library="supply2" deviceset="+5V" device=""/>
 <part name="SUPPLY43" library="supply2" deviceset="GND" device=""/>
+<part name="CRYSTAL" library="con-subd" deviceset="F25" device="VP"/>
+<part name="J1" library="SparkFun-Connectors" deviceset="RASPBERRYPI-40-PIN-GPIO" device="_PTH_NO_SHROUD"/>
+<part name="Q4" library="SparkFun-DiscreteSemi" deviceset="MOSFET-NCH" device="-BSS138" value="220mA/50V/3.5Ω"/>
+<part name="R3" library="resistor" deviceset="R-US_" device="R1206" value="1k"/>
+<part name="SUPPLY44" library="supply2" deviceset="+5V" device=""/>
+<part name="SUPPLY45" library="supply2" deviceset="GND" device=""/>
 </parts>
 <sheets>
@@
 <instance part="SUPPLY34" gate="GND" x="83.82" y="60.96"/>
 <instance part="SUPPLY35" gate="+5V" x="83.82" y="73.66"/>
+<instance part="Q4" gate="NMOS" x="27.94" y="48.26"/>
+<instance part="R3" gate="G$1" x="30.48" y="58.42" rot="R270"/>
+<instance part="SUPPLY44" gate="+5V" x="30.48" y="66.04"/>
+<instance part="SUPPLY45" gate="GND" x="30.48" y="40.64"/>
 </instances>
 <busses>
@@
 <pinref part="C5" gate="G$1" pin="2"/>
 <pinref part="SUPPLY34" gate="GND" pin="GND"/>
+</segment>
+<segment>
+<pinref part="Q4" gate="NMOS" pin="S"/>
+<pinref part="SUPPLY45" gate="GND" pin="GND"/>
 </segment>
 </net>
@@
 <pinref part="C5" gate="G$1" pin="1"/>
 <pinref part="SUPPLY35" gate="+5V" pin="+5V"/>
+</segment>
+<segment>
+<pinref part="R3" gate="G$1" pin="1"/>
+<pinref part="SUPPLY44" gate="+5V" pin="+5V"/>
 </segment>
 </net>
@@
 <wire x1="129.54" y1="17.78" x2="124.46" y2="17.78" width="0.1524" layer="91"/>
 <label x="124.46" y="17.78" size="1.778" layer="95" rot="R180"/>
+</segment>
+<segment>
+<pinref part="Q4" gate="NMOS" pin="G"/>
+<wire x1="22.86" y1="45.72" x2="17.78" y2="45.72" width="0.1524" layer="91"/>
+<label x="17.78" y="45.72" size="1.778" layer="95" rot="R180"/>
 </segment>
 </net>
@@
 <pinref part="IC1" gate="G$1" pin="BW"/>
 <pinref part="R2" gate="G$1" pin="1"/>
+</segment>
+</net>
+<net name="N$11" class="0">
+<segment>
+<pinref part="IC2" gate="A" pin="TR"/>
+<wire x1="50.8" y1="53.34" x2="30.48" y2="53.34" width="0.1524" layer="91"/>
+<pinref part="Q4" gate="NMOS" pin="D"/>
+<pinref part="R3" gate="G$1" pin="2"/>
+<junction x="30.48" y="53.34"/>
 </segment>
 </net>
@@
 <instance part="SUPPLY40" gate="GND" x="53.34" y="50.8"/>
 <instance part="SUPPLY41" gate="+24V" x="73.66" y="83.82"/>
+<instance part="CRYSTAL" gate="-1" x="20.32" y="25.4"/>
 </instances>
 <busses>
@@
 </nets>
 </sheet>
+<sheet>
+<description>Raspberry Pi</description>
+<plain>
+</plain>
+<instances>
+<instance part="J1" gate="G$1" x="53.34" y="58.42"/>
+</instances>
+<busses>
+</busses>
+<nets>
+</nets>
+</sheet>

Commit message: Adding crystal
Parts:
- added C7: 10uF, resistor:C-EUC1206
- added PPSOUT1: BU-SMA-V, con-coax:BU-SMA-V
- added Q5: 35A/25V/8.5mΩ, SparkFun-DiscreteSemi:MOSFET-NCH-FDD8780
- added U$8: MIC5014, FRC696:MIC5014
Connections:
- new net CRYSTAL_EFC: CRYSTAL.5
- new net CRYSTAL_HEAT_EN: U$5.INPUT
- new net CRYSTAL_HEAT_IMON: U$2.VOUT
- new net CRYSTAL_LOGIC: CRYSTAL.15, Q5.S, U$8.SOURCE
- new net CRYSTAL_LOGIC_EN: U$8.INPUT
- new net CRYSTAL_OUT: CRYSTAL.1, PPSOUT1.1
- new net CRYSTAL_OVEN_MON: CRYSTAL.9
- new net N$14: Q5.G, U$8.GATE
- net +24V: now also C7.1, Q5.D, U$8.V+
- net +5V: now also J1.5V@2, J1.5V@4
- net CRYSTAL_HEAT: now also CRYSTAL.10, CRYSTAL.11, CRYSTAL.22, CRYSTAL.23
- net GND: now also C7.2, CRYSTAL.12, CRYSTAL.13, CRYSTAL.14, CRYSTAL.16, CRYSTAL.17, CRYSTAL.2, CRYSTAL.24, CRYSTAL.25, CRYSTAL.3, CRYSTAL.4, J1.GND@14, J1.GND@20, J1.GND@25, J1.GND@30, J1.GND@34, J1.GND@39, J1.GND@6, J1.GND@9, PPSOUT1.2, U$8.GND
